File: Pocket 2.66.kicad_sch (KiCad schematic)
At the start: 74 parts, among them P1 USB-TYPE-C-018, P3 FPC-05F-24PH20, P4 HX-1.25-2AWB, Q1 AO3401-ED, Q2 AO3400, SW1 TS-24CA-S16, SW2 TS-24CA-S16, SW3 TS-24CA-S16, U1 ESP32-C3-MINI-1-N4, U2 LCK-TF-027H37508-WLG, U3 GX4054, U4 GS2019-33TR5, U5 STC3115AIQT, U6 ESD-USB

Commit message: Start of layout with ESP32-C3 mini module
Co-Authored-By: Claude Sonnet 4.6 <noreply@anthropic.com>
Parts:
- removed D4: RED, LCSC:C2286_LED0603-RD, symbol LCSC Global:LED R 0603
- removed P1: USB-TYPE-C-018, LCSC:C2927038_USB-C_SMD-TYPE-C-31-M-12, symbol LCSC Global:USB-TYPE-C-018
- removed P3: FPC-05F-24PH20, LCSC:C2856805_FPC-SMD_24P-P0_50_FPC-05F-24PH20, symbol LCSC Global:FPC-05F-24PH20
- removed P4: HX-1.25-2AWB, LCSC:C52016406_CONN-SMD_2P-P1_25_HX-1_25-2AWB, symbol LCSC Global:picoblade 2-pin
- removed U2: LCK-TF-027H37508-WLG, LCSC:C50380692_TF-SMD_HYCW104-TF08-375B, symbol LCSC Global:LCK-TF-027H37508-WLG
- added D4: LED Yel Side, LCSC:C52675985_LED_Side, symbol LCSC Global:LED Yel Side
- added P1: TYPE-C 16P CB1.6 073, LCSC:C2906290_USB-C-SMD_SHOU_TYPE-C-16P-CB1_6, symbol LCSC Global:TYPE-C_16P_CB1_6_073
- added P2: FPC-24-pin, LCSC:C324726_FFC-SMD_24P-P0_50_FH34SRJ-24S-0_5SH, symbol LCSC Global:FH34SRJ-24S-0_5SH(50)
- added U2: MLD-TF PUSH-H18, LCSC:C52750848_SD-SMD_MLD-TF-PUSH-H18, symbol LCSC Global:micro-SD card slot
- added VBAT1, VBAT2: TestPoint, TestPoint:TestPoint_Pad_D1.0mm, symbol Connector:TestPoint
- C30, C31, R10, R20, R21, R22, R23, R24, R5, R8, R9: JLC Type (none) -> Basic
- L1, SW1, SW2, SW3, U1, U3, U4, U5: JLC Type (none) -> Extended
- U6: JLC Type (none) -> Promotional
Connections:
- net 3V3: now also P2.15, P2.16, U2.4 (VDD)
- net BUSY: now also P2.9
- net CC1: now also P1.A5 (CC1)
- net CC2: now also P1.B5 (CC2)
- net CHRG: now also D4.1 (K)
- net DAT1: now also U2.8 (DAT1)
- net DAT2: now also U2.1 (DAT2)
- net DIS_CS: now also P2.12
- net DIS_DC: now also P2.11
- net DIS_RS: now also P2.10
- net GDR: now also P2.2
- net GND: now also P1.0 (SH), P1.1 (SH), P1.2 (SH), P1.3 (SH), P1.A1 (GND), P1.A12 (GND), P1.B1 (GND), P1.B12 (GND), P2.17, P2.25, P2.26, P2.8, U2.10 (EH), U2.11 (EH), U2.12 (EH), U2.13 (EH), U2.6 (VSS)
- net MISO: now also U2.7 (DAT0)
- net MOSI: now also P2.14, U2.3 (CMD)
- net RESE: now also P2.3
- net SCK: now also P2.13, U2.5 (CLX)
- net SD_CS: now also U2.2 (CD/DAT3)
- net USBD+: now also P1.A6 (DP1), P1.B6 (DP2)
- net USBD-: now also P1.A7 (DN1), P1.B7 (DN2)
- net VBAT: now also VBAT1.1
- net VBAT-: now also VBAT2.1
- net VCOM: now also P2.24
- net VDD_D: now also P2.18
- net VGH: now also P2.21
- net VGL: now also P2.23
- net VGL2: now also P2.4
- net VSH1: now also P2.20
- net VSH2: now also P2.5
- net VSL: now also P2.22
- net VUSB: now also U6.3, P1.A4 (VBUS), P1.A9 (VBUS), P1.B4 (VBUS), P1.B9 (VBUS)
- net BATD: now reaches R19.2, U5.8 (BATD/CD)
- net LTY: now reaches R21.1
- net LTY: now also D4.2 (A)
- no-connect marks 25 -> 23
